Commit message: se hicieron cambios

File: manipulator_description/urdf/manipulator_macro.xacro (robot description, xacro)
@@ -55,5 +55,5 @@
         rpy="0 0 0" />
       <mass
-        value="0.0569176277607128" />
+        value="0.102" />
       <inertia
         ixx="26860"
@@ -171,5 +171,5 @@
         rpy="0 0 0" />
       <mass
-        value="0.0569176277607127" />
+        value="0.102" />
       <inertia
         ixx="26860"
@@ -287,5 +287,5 @@
         rpy="0 0 0" />
       <mass
-        value="0.0569176277607127" />
+        value="0.102" />
       <inertia
         ixx="26860"

File: manipulator_moveit/config/gazebo_manipulator_robot.urdf (robot description, URDF)
Before this commit: robot manipulator_robot, 8 links, 7 joints
Links:
- link link_1: mass 0.0569176277607128 -> 0.102
- link link_3: mass 0.0569176277607127 -> 0.102
- link link_5: mass 0.0569176277607127 -> 0.102

Commit message: Se cambio las inercias del urdf y todo el paquete del moveit con los nuevos cambios

File: manipulator_description/urdf/manipulator_macro.xacro (robot description, xacro)
@@ -8,5 +8,5 @@
         <origin rpy="0.0 0.0 0.0" xyz="0.0 0.0 0.0" />
     </joint>
-  <link
+ <link
     name="base_link">
     <inertial>
@@ -17,10 +17,10 @@
         value="0.391381454473344" />
       <inertia
-        ixx="224200000"
-        ixy="-102530000"
-        ixz="10964000"
-        iyy="935460000"
-        iyz="-533770"
-        izz="777040000" />
+        ixx="0.101795155"
+        ixy="-0.0000106"
+        ixz="-0.000004255"
+        iyy="0.1049705"
+        iyz="-0.0025166"
+        izz="0.113806134" />
     </inertial>
     <visual>
@@ -57,10 +57,10 @@
         value="0.102" />
       <inertia
-        ixx="26860"
-        ixy="525.09"
-        ixz="287.62"
-        iyy="16993"
-        iyz="-523.85"
-        izz="26995" />
+        ixx="0.004708"
+        ixy="0.0000362"
+        ixz="-0.0000863"
+        iyy="0.0034761"
+        iyz="-0.0013745"
+        izz="0.0024097" />
     </inertial>
     <visual>
@@ -115,10 +115,10 @@
         value="0.102283747087815" />
       <inertia
-        ixx="512810000"
-        ixy="108850000"
-        ixz="380"
-        iyy="56237000"
-        iyz="2370"
-        izz="523870000" />
+        ixx="0.125060728"
+        ixy="0.017650428"
+        ixz="0.000000038"
+        iyy="0.0057453"
+        iyz="-0.00000199"
+        izz="0.1262878" />
     </inertial>
     <visual>
@@ -173,10 +173,10 @@
         value="0.102" />
       <inertia
-        ixx="26860"
-        ixy="525.09"
-        ixz="287.62"
-        iyy="16993"
-        iyz="-523.85"
-        izz="26995" />
+        ixx="0.004708"
+        ixy="0.0000362"
+        ixz="-0.0000863"
+        iyy="0.0034761"
+        iyz="-0.0013745"
+        izz="0.0024097" />
     </inertial>
     <visual>
@@ -231,10 +231,10 @@
         value="0.105070462984835" />
       <inertia
-        ixx="1573100000"
-        ixy="195670000"
-        ixz="40"
-        iyy="51205000"
-        iyz="1350"
-        izz="1589800000"/>
+        ixx="0.1573144"
+        ixy="0.0195671"
+        ixz="0.0000000040"
+        iyy="0.0051205"
+        iyz="0.0000001350"
+        izz="0.1589789"/>
     </inertial>
     <visual>
@@ -287,12 +287,12 @@
         rpy="0 0 0" />
       <mass
-        value="0.102" />
-      <inertia
-        ixx="26860"
-        ixy="525.09"
-        ixz="287.62"
-        iyy="16993"
-        iyz="-523.85"
-        izz="26995" />
+        value="0.0982" />
+      <inertia
+        ixx="0.004708"
+        ixy="0.0000362"
+        ixz="-0.0000863"
+        iyy="0.0034761"
+        iyz="-0.0013745"
+        izz="0.0024097" />
     </inertial>
     <visual>
@@ -347,10 +347,10 @@
         value="0.00405886351711359" />
       <inertia
-        ixx="3316900"
-        ixy="-10"
+        ixx="0.0000873"
+        ixy="0"
         ixz="0"
-        iyy="3315500"
+        iyy="0.0000873"
         iyz="0"
-        izz="185540" />
+        izz="0.0000237" />
     </inertial>
     <visual>

File: manipulator_moveit/config/gazebo_manipulator_robot.urdf (robot description, URDF)
Before this commit: robot manipulator_robot, 8 links, 7 joints
Links:
- link link_5: mass 0.102 -> 0.0982

Commit message: se realizo de nuevo el moveit con el nuevo urdf creado para el marcador

File: manipulator_description/urdf/manipulator_macro.xacro (robot description, xacro)
@@ -8,5 +8,5 @@
         <origin rpy="0.0 0.0 0.0" xyz="0.0 0.0 0.0" />
     </joint>
- <link
+  <link
     name="base_link">
     <inertial>
@@ -342,15 +342,15 @@
     <inertial>
       <origin
-        xyz="1.27935106952748E-10 -1.49986290117875E-05 0.0091913137007949"
-        rpy="0 0 0" />
-      <mass
-        value="0.00405886351711359" />
-      <inertia
-        ixx="0.0000873"
-        ixy="0"
+        xyz="2.13388832944876E-08 -5.97864488471878E-08 0.0686884907670908"
+        rpy="0 0 0" />
+      <mass
+        value="0.0340927901942582" />
+      <inertia
+        ixx="133722.55E-9"
+        ixy="0.01E-9"
         ixz="0"
-        iyy="0.0000873"
-        iyz="0"
-        izz="0.0000237" />
+        iyy="133722.55E-9"
+        iyz="-0.05E-9"
+        izz="1130.56E-9" />
     </inertial>
     <visual>

File: manipulator_moveit/config/gazebo_manipulator_robot.urdf (robot description, URDF)
Before this commit: robot manipulator_robot, 8 links, 7 joints
Links:
- link link_6: mass 0.00405886351711359 -> 0.0340927901942582
