Commit message: URDF actualizados

File: manipulator_description/urdf/manipulator.urdf (robot description, URDF)
Before this commit: robot manipulator_main, 8 links, 7 joints
Links:
- link base_link: mass 0.14032 -> 0.391381454473344
- link link_1: mass 0.05168 -> 0.0569176277607128
- link link_2: mass 0.10228 -> 0.102283747087815
- link link_3: mass 0.05168 -> 0.0569176277607127
- link link_4: mass 0.10507 -> 0.105070462984835
- link link_5: mass 0.05168 -> 0.0569176277607127
- link link_6: mass 0.006005 -> 0.00405886351711359; geometry collision mesh filename=package://manipulator_description/meshes/link_6.STL; visual mesh filename=package://manipulator_description/meshes/link_6.STL
Joints:
- joint joint_1: limit lower=0 upper=0 effort=0 velocity=0 -> lower=-1.57 upper=1.57 effort=300 velocity=3; origin xyz=0 0 0.039971 rpy=0 0 0 -> xyz=0 0 0.0688 rpy=0 0 3.1416; type continuous -> revolute
- joint joint_2: limit lower=0 upper=0 effort=0 velocity=0 -> lower=-0.78 upper=0.78 effort=300 velocity=3; origin xyz=0.024 0.019 0.0090292 rpy=-1.5708 -0.0070881 0 -> xyz=0 -0.024 0.02 rpy=1.5708 0 -1.5708; type continuous -> revolute
- joint joint_3: limit lower=0 upper=0 effort=0 velocity=0 -> lower=-1.15 upper=2 effort=300 velocity=3; origin xyz=-0.024 -0.195 -0.019 rpy=3.1416 0 0 -> xyz=-0.024 0.195 0 rpy=0 0 3.1416; type continuous -> revolute
- joint joint_4: axis 0 0 1 -> 0 1 0; limit lower=0 upper=0 effort=0 velocity=0 -> lower=-3.14 upper=3.14 effort=200 velocity=3; origin xyz=0.019 0.024 0 rpy=3.1416 1.5656 3.1345 -> xyz=-0.019 -0.024 0 rpy=0 0 1.5708; type continuous -> revolute
- joint joint_5: axis 0 0 1 -> 1 0 0; limit lower=0 upper=0 effort=0 velocity=0 -> lower=-1.15 upper=2 effort=200 velocity=3; origin xyz=-0.00099824 -0.022521 0.20866 rpy=-1.57 3.14  1.57 -> xyz=0.024 0.2085 0 rpy=0 -1.5708 0; type continuous -> revolute
- joint joint_6: limit lower=0 upper=0 effort=0 velocity=0 -> lower=-3.14 upper=3.14 effort=200 velocity=3; origin xyz=0.01883 0.02412 0 rpy=-1.5708 1.5312 -1.5637 -> xyz=0 0.024 -0.019 rpy=3.1416 0 -1.5354; type continuous -> revolute

File: manipulator_description/urdf/manipulator_macro.xacro (robot description, xacro)
@@ -1,11 +1,19 @@
 <?xml version="1.0"?>
 <robot xmlns:xacro="http://wiki.ros.org/xacro">
-  <!-- Links del robot -->
-    <link name="base_link">
-    <inertial>
-      <origin
-        xyz="0.001243 9.6973E-06 0.018348" rpy="0 0 0" />
-      <mass
-        value="0.14032" />
+  <!-- Fix robot to Gazebo world -->
+    <link name="world" />
+    <joint name="world-base_link-fixed" type="fixed">
+        <parent link="world" />
+        <child link="base_link" />
+        <origin rpy="0.0 0.0 0.0" xyz="0.0 0.0 0.0" />
+    </joint>
+  <link
+    name="base_link">
+    <inertial>
+      <origin
+        xyz="5.34102915090225E-06 0.00149611119634718 0.027324411040906"
+        rpy="0 0 0" />
+      <mass
+        value="0.391381454473344" />
       <inertia
         ixx="224200000"
@@ -18,5 +26,6 @@
     <visual>
       <origin
-        xyz="0 0 0" rpy="0 0 0" />
+        xyz="0 0 0"
+        rpy="0 0 0" />
       <geometry>
         <mesh
@@ -26,10 +35,11 @@
         name="">
         <color
-          rgba="0.69804 0.69804 0.69804 1" />
-      </material>
-    </visual>
-    <collision>
-      <origin
-        xyz="0 0 0" rpy="0 0 0" />
+          rgba="0.698039215686274 0.698039215686274 0.698039215686274 1" />
+      </material>
+    </visual>
+    <collision>
+      <origin
+        xyz="0 0 0"
+        rpy="0 0 0" />
       <geometry>
         <mesh
@@ -38,10 +48,12 @@
     </collision>
   </link>
-  <link name="link_1">
-    <inertial>
-      <origin
-        xyz="0.012 -0.00063149 0.0083979" rpy="0 0 0" />
-      <mass
-        value="0.05168" />
+  <link
+    name="link_1">
+    <inertial>
+      <origin
+        xyz="0.000495971250250978 -0.0119998499605218 0.0204959033777655"
+        rpy="0 0 0" />
+      <mass
+        value="0.0569176277607128" />
       <inertia
         ixx="26860"
@@ -54,5 +66,6 @@
     <visual>
       <origin
-        xyz="0 0 0" rpy="0 0 0" />
+        xyz="0 0 0"
+        rpy="0 0 0" />
       <geometry>
         <mesh
@@ -62,10 +75,11 @@
         name="">
         <color
-          rgba="0.79216 0.81961 0.93333 1" />
-      </material>
-    </visual>
-    <collision>
-      <origin
-        xyz="0 0 0" rpy="0 0 0" />
+          rgba="0.752941176470588 0.752941176470588 0.752941176470588 1" />
+      </material>
+    </visual>
+    <collision>
+      <origin
+        xyz="0 0 0"
+        rpy="0 0 0" />
       <geometry>
         <mesh
@@ -74,10 +88,30 @@
     </collision>
   </link>
-    <link name="link_2">
-    <inertial>
-      <origin
-        xyz="-0.011752 -0.099865 -0.019" rpy="0 0 0" />
-      <mass
-        value="0.10228" />
+  <joint
+    name="joint_1"
+    type="revolute">
+    <origin
+      xyz="0 0 0.0688"
+      rpy="0 0 3.1416" />
+    <parent
+      link="base_link" />
+    <child
+      link="link_1" />
+    <axis
+      xyz="0 0 1" />
+    <limit
+      lower="-1.57"
+      upper="1.57"
+      effort="300"
+      velocity="3" />
+  </joint>
+  <link
+    name="link_2">
+    <inertial>
+      <origin
+        xyz="-0.0117522388524779 0.099865169344438 3.09623365025784E-07"
+        rpy="0 0 0" />
+      <mass
+        value="0.102283747087815" />
       <inertia
         ixx="512810000"
@@ -90,5 +124,6 @@
     <visual>
       <origin
-        xyz="0 0 0" rpy="0 0 0" />
+        xyz="0 0 0"
+        rpy="0 0 0" />
       <geometry>
         <mesh
@@ -98,10 +133,11 @@
         name="">
         <color
-          rgba="0.69804 0.69804 0.69804 1" />
-      </material>
-    </visual>
-    <collision>
-      <origin
-        xyz="0 0 0" rpy="0 0 0" />
+          rgba="0.698039215686274 0.698039215686274 0.698039215686274 1" />
+      </material>
+    </visual>
+    <collision>
+      <origin
+        xyz="0 0 0"
+        rpy="0 0 0" />
       <geometry>
         <mesh
@@ -110,10 +146,30 @@
     </collision>
   </link>
-  <link name="link_3">
-    <inertial>
-      <origin
-        xyz="0.00063139 0.012 -0.00063149" rpy="0 0 0" />
-      <mass
-        value="0.05168" />
+  <joint
+    name="joint_2"
+    type="revolute">
+    <origin
+      xyz="0 -0.024 0.02"
+      rpy="1.5708 0 -1.5708" />
+    <parent
+      link="link_1" />
+    <child
+      link="link_2" />
+    <axis
+      xyz="0 0 1" />
+    <limit
+      lower="-0.78"
+      upper="0.78"
+      effort="300"
+      velocity="3" />
+  </joint>
+  <link
+    name="link_3">
+    <inertial>
+      <origin
+        xyz="0.000495971402698712 -0.0119998503185919 0.000495878377765541"
+        rpy="0 0 0" />
+      <mass
+        value="0.0569176277607127" />
       <inertia
         ixx="26860"
@@ -126,5 +182,6 @@
     <visual>
       <origin
-        xyz="0 0 0" rpy="0 0 0" />
+        xyz="0 0 0"
+        rpy="0 0 0" />
       <geometry>
         <mesh
@@ -134,10 +191,11 @@
         name="">
         <color
-          rgba="0.79216 0.81961 0.93333 1" />
-      </material>
-    </visual>
-    <collision>
-      <origin
-        xyz="0 0 0" rpy="0 0 0" />
+          rgba="0.752941176470588 0.752941176470588 0.752941176470588 1" />
+      </material>
+    </visual>
+    <collision>
+      <origin
+        xyz="0 0 0"
+        rpy="0 0 0" />
       <geometry>
         <mesh
@@ -146,10 +204,30 @@
     </collision>
   </link>
-  <link name="link_4">
-    <inertial>
-      <origin
-        xyz="-0.00050964 -0.011144 0.1062" rpy="0 0 0" />
-      <mass
-        value="0.10507" />
+  <joint
+    name="joint_3"
+    type="revolute">
+    <origin
+      xyz="-0.024 0.195 0"
+      rpy="0 0 3.1416" />
+    <parent
+      link="link_2" />
+    <child
+      link="link_3" />
+    <axis
+      xyz="0 0 1" />
+    <limit
+      lower="-1.15"
+      upper="2"
+      effort="300"
+      velocity="3" />
+  </joint>
+  <link
+    name="link_4">
+    <inertial>
+      <origin
+        xyz="0.0118962971363374 0.106115026058573 4.33165647320523E-07"
+        rpy="0 0 0" />
+      <mass
+        value="0.105070462984835" />
       <inertia
         ixx="1573100000"
@@ -158,9 +236,10 @@
         iyy="51205000"
         iyz="1350"
-        izz="1589800000" />
-    </inertial>
-    <visual>
-      <origin
-        xyz="0 0 0" rpy="0 0 0" />
+        izz="1589800000"/>
+    </inertial>
+    <visual>
+      <origin
+        xyz="0 0 0"
+        rpy="0 0 0" />
       <geometry>
         <mesh
@@ -170,10 +249,11 @@
         name="">
         <color
-          rgba="0.69804 0.69804 0.69804 1" />
-      </material>
-    </visual>
-    <collision>
-      <origin
-        xyz="0 0 0" rpy="0 0 0" />
+          rgba="0.698039215686274 0.698039215686274 0.698039215686274 1" />
+      </material>
+    </visual>
+    <collision>
+      <origin
+        xyz="0 0 0"
+        rpy="0 0 0" />
       <geometry>
         <mesh
@@ -182,10 +262,30 @@
     </collision>
   </link>
-  <link name="link_5">
-    <inertial>
-      <origin
-        xyz="0.00054632 0.012004 -0.00063149" rpy="0 0 0" />
-      <mass
-        value="0.05168" />
+  <joint
+    name="joint_4"
+    type="revolute">
+    <origin
+      xyz="-0.019 -0.024 0"
+      rpy="0 0 1.5708" />
+    <parent
+      link="link_3" />
+    <child
+      link="link_4" />
+    <axis
+      xyz="0 1 0" />
+    <limit
+      lower="-3.14"
+      upper="3.14"
+      effort="200"
+      velocity="3" />
+  </joint>
+  <link
+    name="link_5">
+    <inertial>
+      <origin
+        xyz="0.000495971250250887 0.0120001503975483 0.000495878530213656"
+        rpy="0 0 0" />
+      <mass
+        value="0.0569176277607127" />
       <inertia
         ixx="26860"
@@ -198,5 +298,6 @@
     <visual>
       <origin
-        xyz="0 0 0" rpy="0 0 0" />
+        xyz="0 0 0"
+        rpy="0 0 0" />
       <geometry>
         <mesh
@@ -206,10 +307,11 @@
         name="">
         <color
-          rgba="0.79216 0.81961 0.93333 1" />
-      </material>
-    </visual>
-    <collision>
-      <origin
-        xyz="0 0 0" rpy="0 0 0" />
+          rgba="0.752941176470588 0.752941176470588 0.752941176470588 1" />
+      </material>
+    </visual>
+    <collision>
+      <origin
+        xyz="0 0 0"
+        rpy="0 0 0" />
       <geometry>
         <mesh
@@ -218,10 +320,30 @@
     </collision>
   </link>
-  <link name="link_6">
-    <inertial>
-      <origin
-        xyz="9.9252E-09 -4.0368E-07 0.018675" rpy="0 0 0" />
-      <mass
-        value="0.006005" />
+  <joint
+    name="joint_5"
+    type="revolute">
+    <origin
+      xyz="0.024 0.2085 0"
+      rpy="0 -1.5708 0" />
+    <parent
+      link="link_4" />
+    <child
+      link="link_5" />
+    <axis
+      xyz="1 0 0" />
+    <limit
+      lower="-1.15"
+      upper="2"
+      effort="200"
+      velocity="3" />
+  </joint>
+  <link
+    name="link_6">
+    <inertial>
+      <origin
+        xyz="1.27935106952748E-10 -1.49986290117875E-05 0.0091913137007949"
+        rpy="0 0 0" />
+      <mass
+        value="0.00405886351711359" />
       <inertia
         ixx="3316900"
@@ -234,94 +356,136 @@
     <visual>
       <origin
-        xyz="0 0 0" rpy="0 0 0" />
-      <geometry>
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
Commit message: Update manipulator.urdf

File: manipulator_description/urdf/manipulator.urdf (robot description, URDF)
Before this commit: robot manipulator, 8 links, 7 joints
Links:
- link link_1: mass 0.0569176277607128 -> 0.102
- link link_3: mass 0.0569176277607127 -> 0.102
- link link_5: mass 0.0569176277607127 -> 0.0982

Commit message: Cambios en el URDF y Meshes

File: manipulator_description/urdf/manipulator.urdf (robot description, URDF)
Before this commit: robot manipulator, 8 links, 7 joints
Links:
- link link_6: mass 0.00405886351711359 -> 0.0340927901942582

Commit message: se hizo el cambio con el URDF arreglado y funciono todo correctamente

File: manipulator_description/urdf/manipulator.urdf (robot description, URDF)
Before this commit: robot manipulator, 8 links, 7 joints
Links:
- link base_link: mass 0.391381454473344 -> 0.399055600639488
- link link_4: mass 0.105070462984835 -> 0.105070462984836
Joints:
- joint joint_1: origin xyz=0 0 0.0688 rpy=0 0 3.1416 -> xyz=0 0 0.07 rpy=0 0 3.14159265358979
- joint joint_2: origin xyz=0 -0.024 0.02 rpy=1.5708 0 -1.5708 -> xyz=0 -0.02 0.02 rpy=1.5707963267949 0 -1.5707963267949
- joint joint_3: origin xyz=-0.024 0.195 0 rpy=0 0 3.1416 -> xyz=-0.02 0.2 0 rpy=0 0 1.5707963267949
- joint joint_4: axis 0 1 0 -> 0 0 1; origin xyz=-0.019 -0.024 0 rpy=0 0 1.5708 -> xyz=0.0200000000000001 -0.02 0 rpy=1.5707963267949 0 0
- joint joint_5: axis 1 0 0 -> 0 0 1; origin xyz=0.024 0.2085 0 rpy=0 -1.5708 0 -> xyz=-0.0200000000000001 0 0.21 rpy=-1.5707963267949 0 0
- joint joint_6: origin xyz=0 0.024 -0.019 rpy=3.1416 0 -1.5354 -> xyz=-0.04 -0.02 0 rpy=1.5707963267949 0 -1.5707963267949

File: manipulator_description/urdf/manipulator_macro.xacro (robot description, xacro)
@@ -12,8 +12,8 @@
     <inertial>
       <origin
-        xyz="5.34102915090225E-06 0.00149611119634718 0.027324411040906"
-        rpy="0 0 0" />
-      <mass
-        value="0.391381454473344" />
+        xyz="5.34102915090199E-06 0.00149611119634719 0.027324411040906"
+        rpy="0 0 0" />
+      <mass
+        value="0.399055600639488" />
       <inertia
         ixx="0.101795155"
@@ -35,5 +35,5 @@
         name="">
         <color
-          rgba="0.698039215686274 0.698039215686274 0.698039215686274 1" />
+          rgba="0.0549 0.4 0.3333 1.0"/>
       </material>
     </visual>
@@ -52,5 +52,5 @@
     <inertial>
       <origin
-        xyz="0.000495971250250978 -0.0119998499605218 0.0204959033777655"
+        xyz="0.000495971250250975 -0.0119998499605218 0.0192958783777655"
         rpy="0 0 0" />
       <mass
@@ -75,5 +75,5 @@
         name="">
         <color
-          rgba="0.752941176470588 0.752941176470588 0.752941176470588 1" />
+          rgba="0.09019 0.12549 0.164706 1.0"/>
       </material>
     </visual>
@@ -92,6 +92,6 @@
     type="revolute">
     <origin
-      xyz="0 0 0.0688"
-      rpy="0 0 3.1416" />
+      xyz="0 0 0.07"
+      rpy="0 0 3.14159265358979" />
     <parent
       link="base_link" />
@@ -110,5 +110,5 @@
     <inertial>
       <origin
-        xyz="-0.0117522388524779 0.099865169344438 3.09623365025784E-07"
+        xyz="-0.00775223885247785 0.0986651693444381 3.09623365033344E-07"
         rpy="0 0 0" />
       <mass
@@ -133,5 +133,5 @@
         name="">
         <color
-          rgba="0.698039215686274 0.698039215686274 0.698039215686274 1" />
+          rgba="0.1804 0.8 0.4431 1.0"/>
       </material>
     </visual>
@@ -150,6 +150,6 @@
     type="revolute">
     <origin
-      xyz="0 -0.024 0.02"
-      rpy="1.5708 0 -1.5708" />
+      xyz="0 -0.02 0.02"
+      rpy="1.5707963267949 0 -1.5707963267949" />
     <parent
       link="link_1" />
@@ -168,5 +168,5 @@
     <inertial>
       <origin
-        xyz="0.000495971402698712 -0.0119998503185919 0.000495878377765541"
+        xyz="0.0057998503185917 0.000495971402698678 0.000495878377765527"
         rpy="0 0 0" />
       <mass
@@ -191,5 +191,5 @@
         name="">
         <color
-          rgba="0.752941176470588 0.752941176470588 0.752941176470588 1" />
+          rgba="0.09019 0.12549 0.164706 1.0"/>
       </material>
     </visual>
@@ -208,6 +208,6 @@
     type="revolute">
     <origin
-      xyz="-0.024 0.195 0"
-      rpy="0 0 3.1416" />
+      xyz="-0.02 0.2 0"
+      rpy="0 0 1.5707963267949" />
     <parent
       link="link_2" />
@@ -226,8 +226,8 @@
     <inertial>
       <origin
-        xyz="0.0118962971363374 0.106115026058573 4.33165647320523E-07"
-        rpy="0 0 0" />
-      <mass
-        value="0.105070462984835" />
+        xyz="-0.0140962967782675 4.33165647224752E-07 0.105115025906125"
+        rpy="0 0 0" />
+      <mass
+        value="0.105070462984836" />
       <inertia
         ixx="0.1573144"
@@ -249,5 +249,5 @@
         name="">
         <color
-          rgba="0.698039215686274 0.698039215686274 0.698039215686274 1" />
+          rgba="0.1804 0.8 0.4431 1.0"/>
       </material>
     </visual>
@@ -266,6 +266,6 @@
     type="revolute">
     <origin
-      xyz="-0.019 -0.024 0"
-      rpy="0 0 1.5708" />
+      xyz="0.0200000000000001 -0.02 0"
+      rpy="1.5707963267949 0 0" />
     <parent
       link="link_3" />
@@ -273,5 +273,5 @@
       link="link_4" />
     <axis
-      xyz="0 1 0" />
+      xyz="0 0 1" />
     <limit
       lower="-3.14"
@@ -284,5 +284,5 @@
     <inertial>
       <origin
-        xyz="0.000495971250250887 0.0120001503975483 0.000495878530213656"
+        xyz="-0.00570412111171636 -0.00950015024510067 0.000495971250250971"
         rpy="0 0 0" />
       <mass
@@ -307,5 +307,5 @@
         name="">
         <color
-          rgba="0.752941176470588 0.752941176470588 0.752941176470588 1" />
+          rgba="0.09019 0.12549 0.164706 1.0"/>
       </material>
     </visual>
@@ -324,6 +324,6 @@
     type="revolute">
     <origin
-      xyz="0.024 0.2085 0"
-      rpy="0 -1.5708 0" />
+      xyz="-0.0200000000000001 0 0.21"
+      rpy="-1.5707963267949 0 0" />
     <parent
       link="link_4" />
@@ -331,5 +331,5 @@
       link="link_5" />
     <axis
-      xyz="1 0 0" />
+      xyz="0 0 1" />
     <limit
       lower="-1.15"
@@ -342,5 +342,5 @@
     <inertial>
       <origin
-        xyz="2.13388832944876E-08 -5.97864488471878E-08 0.0686884907670908"
+        xyz="0.00150005999207131 2.13388833428252E-08 0.0547308096922248"
         rpy="0 0 0" />
       <mass
@@ -365,5 +365,5 @@
         name="">
         <color
-          rgba="1 0.549019607843137 0 1" />
+          rgba="0.729411764705882 0.356862745098039 0.0235294117647059 1" />
       </material>
     </visual>
@@ -382,6 +382,6 @@
     type="revolute">
     <origin
-      xyz="0 0.024 -0.019"
-      rpy="3.1416 0 -1.5354" />
+      xyz="-0.04 -0.02 0"
+      rpy="1.5707963267949 0 -1.5707963267949" />
     <parent
       link="link_5" />

File: manipulator_moveit/config/gazebo_manipulator_robot.urdf (robot description, URDF)
Before this commit: robot manipulator_robot, 8 links, 7 joints
Links:
- link base_link: mass 0.391381454473344 -> 0.399055600639488
- link link_4: mass 0.105070462984835 -> 0.105070462984836
Joints:
- joint joint_1: origin xyz=0 0 0.0688 rpy=0 0 3.1416 -> xyz=0 0 0.07 rpy=0 0 3.14159265358979
- joint joint_2: origin xyz=0 -0.024 0.02 rpy=1.5708 0 -1.5708 -> xyz=0 -0.02 0.02 rpy=1.5707963267949 0 -1.5707963267949
- joint joint_3: origin xyz=-0.024 0.195 0 rpy=0 0 3.1416 -> xyz=-0.02 0.2 0 rpy=0 0 1.5707963267949
- joint joint_4: axis 0 1 0 -> 0 0 1; origin xyz=-0.019 -0.024 0 rpy=0 0 1.5708 -> xyz=0.0200000000000001 -0.02 0 rpy=1.5707963267949 0 0
- joint joint_5: axis 1 0 0 -> 0 0 1; origin xyz=0.024 0.2085 0 rpy=0 -1.5708 0 -> xyz=-0.0200000000000001 0 0.21 rpy=-1.5707963267949 0 0
- joint joint_6: origin xyz=0 0.024 -0.019 rpy=3.1416 0 -1.5354 -> xyz=-0.04 -0.02 0 rpy=1.5707963267949 0 -1.5707963267949
