Commit message: Cambio de nombre de paquetes

File: manipulator_description/urdf/manipulator.urdf (robot description, URDF)
Before this commit: robot manipulator, 8 links, 7 joints
Links:
- link base_link: geometry collision mesh filename=package://archie_description/meshes/base_link.STL; visual mesh filename=package://archie_description/meshes/base_link.STL
- link link_1: geometry collision mesh filename=package://archie_description/meshes/link_1.STL; visual mesh filename=package://archie_description/meshes/link_1.STL
- link link_2: geometry collision mesh filename=package://archie_description/meshes/link_2.STL; visual mesh filename=package://archie_description/meshes/link_2.STL
- link link_3: geometry collision mesh filename=package://archie_description/meshes/link_3.STL; visual mesh filename=package://archie_description/meshes/link_3.STL
- link link_4: geometry collision mesh filename=package://archie_description/meshes/link_4.STL; visual mesh filename=package://archie_description/meshes/link_4.STL
- link link_5: geometry collision mesh filename=package://archie_description/meshes/link_5.STL; visual mesh filename=package://archie_description/meshes/link_5.STL
- link link_6: geometry collision mesh filename=package://archie_description/meshes/link_6.STL; visual mesh filename=package://archie_description/meshes/link_6.STL

File: manipulator_description/urdf/manipulator.xacro (robot description, xacro)
@@ -1,4 +1,4 @@
 <?xml version="1.0"?>
 <robot name="manipulator_robot" xmlns:xacro="http://wiki.ros.org/xacro">
-  <xacro:include filename="$(find manipulator_description)/urdf/manipulator_macro.xacro" />
+  <xacro:include filename="$(find archie_description)/urdf/manipulator_macro.xacro" />
 </robot>

File: manipulator_description/urdf/manipulator_macro.xacro (robot description, xacro)
@@ -30,5 +30,5 @@
       <geometry>
         <mesh
-          filename="package://manipulator_description/meshes/base_link.STL" />
+          filename="package://archie_description/meshes/base_link.STL" />
       </geometry>
       <material
@@ -44,5 +44,5 @@
       <geometry>
         <mesh
-          filename="package://manipulator_description/meshes/base_link.STL" />
+          filename="package://archie_description/meshes/base_link.STL" />
       </geometry>
     </collision>
@@ -70,5 +70,5 @@
       <geometry>
         <mesh
-          filename="package://manipulator_description/meshes/link_1.STL" />
+          filename="package://archie_description/meshes/link_1.STL" />
       </geometry>
       <material
@@ -84,5 +84,5 @@
       <geometry>
         <mesh
-          filename="package://manipulator_description/meshes/link_1.STL" />
+          filename="package://archie_description/meshes/link_1.STL" />
       </geometry>
     </collision>
@@ -128,5 +128,5 @@
       <geometry>
         <mesh
-          filename="package://manipulator_description/meshes/link_2.STL" />
+          filename="package://archie_description/meshes/link_2.STL" />
       </geometry>
       <material
@@ -142,5 +142,5 @@
       <geometry>
         <mesh
-          filename="package://manipulator_description/meshes/link_2.STL" />
+          filename="package://archie_description/meshes/link_2.STL" />
       </geometry>
     </collision>
@@ -186,5 +186,5 @@
       <geometry>
         <mesh
-          filename="package://manipulator_description/meshes/link_3.STL" />
+          filename="package://archie_description/meshes/link_3.STL" />
       </geometry>
       <material
@@ -200,5 +200,5 @@
       <geometry>
         <mesh
-          filename="package://manipulator_description/meshes/link_3.STL" />
+          filename="package://archie_description/meshes/link_3.STL" />
       </geometry>
     </collision>
@@ -244,5 +244,5 @@
       <geometry>
         <mesh
-          filename="package://manipulator_description/meshes/link_4.STL" />
+          filename="package://archie_description/meshes/link_4.STL" />
       </geometry>
       <material
@@ -258,5 +258,5 @@
       <geometry>
         <mesh
-          filename="package://manipulator_description/meshes/link_4.STL" />
+          filename="package://archie_description/meshes/link_4.STL" />
       </geometry>
     </collision>
@@ -302,5 +302,5 @@
       <geometry>
         <mesh
-          filename="package://manipulator_description/meshes/link_5.STL" />
+          filename="package://archie_description/meshes/link_5.STL" />
       </geometry>
       <material
@@ -316,5 +316,5 @@
       <geometry>
         <mesh
-          filename="package://manipulator_description/meshes/link_5.STL" />
+          filename="package://archie_description/meshes/link_5.STL" />
       </geometry>
     </collision>
@@ -360,5 +360,5 @@
       <geometry>
         <mesh
-          filename="package://manipulator_description/meshes/link_6.STL" />
+          filename="package://archie_description/meshes/link_6.STL" />
       </geometry>
       <material
@@ -374,5 +374,5 @@
       <geometry>
         <mesh
-          filename="package://manipulator_description/meshes/link_6.STL" />
+          filename="package://archie_description/meshes/link_6.STL" />
       </geometry>
     </collision>

File: manipulator_description/urdf/manipulator_without_pen.urdf (robot description, URDF)
Before this commit: robot manipulator_without_gripper, 7 links, 6 joints
Links:
- link base_link: geometry collision mesh filename=package://archie_description/meshes/base_link.STL; visual mesh filename=package://archie_description/meshes/base_link.STL
- link link_1: geometry collision mesh filename=package://archie_description/meshes/link_1.STL; visual mesh filename=package://archie_description/meshes/link_1.STL
- link link_2: geometry collision mesh filename=package://archie_description/meshes/link_2.STL; visual mesh filename=package://archie_description/meshes/link_2.STL
- link link_3: geometry collision mesh filename=package://archie_description/meshes/link_3.STL; visual mesh filename=package://archie_description/meshes/link_3.STL
- link link_4: geometry collision mesh filename=package://archie_description/meshes/link_4.STL; visual mesh filename=package://archie_description/meshes/link_4.STL
- link link_5: geometry collision mesh filename=package://archie_description/meshes/link_5.STL; visual mesh filename=package://archie_description/meshes/link_5.STL
- link link_6: geometry collision mesh filename=package://archie_description/meshes/link_62.STL; visual mesh filename=package://archie_description/meshes/link_62.STL

File: manipulator_moveit/config/gazebo_manipulator_robot.urdf (robot description, URDF)
Before this commit: robot manipulator_robot, 8 links, 7 joints
Links:
- link base_link: geometry collision mesh filename=package://archie_description/meshes/base_link.STL; visual mesh filename=package://archie_description/meshes/base_link.STL
- link link_1: geometry collision mesh filename=package://archie_description/meshes/link_1.STL; visual mesh filename=package://archie_description/meshes/link_1.STL
- link link_2: geometry collision mesh filename=package://archie_description/meshes/link_2.STL; visual mesh filename=package://archie_description/meshes/link_2.STL
- link link_3: geometry collision mesh filename=package://archie_description/meshes/link_3.STL; visual mesh filename=package://archie_description/meshes/link_3.STL
- link link_4: geometry collision mesh filename=package://archie_description/meshes/link_4.STL; visual mesh filename=package://archie_description/meshes/link_4.STL
- link link_5: geometry collision mesh filename=package://archie_description/meshes/link_5.STL; visual mesh filename=package://archie_description/meshes/link_5.STL
- link link_6: geometry collision mesh filename=package://archie_description/meshes/link_6.STL; visual mesh filename=package://archie_description/meshes/link_6.STL
