Commit message: Nuevo URDF

File: manipulator_final2/urdf/manipulator_final2.urdf (robot description, URDF)
Before this commit: robot manipulator_final2, 7 links, 6 joints
Links:
- link base_link: mass 0.39906 -> 0.399055600639488
- link link_1: mass 0.056918 -> 0.0569176277607128
- link link_2: mass 0.10228 -> 0.102283747087815
Joints:
- joint joint_1: origin xyz=0 0 0.0688 rpy=0 0 3.1416 -> xyz=0 0 0.07 rpy=0 0 3.14159265358979
- joint joint_2: origin xyz=0 -0.024 0.02 rpy=1.5708 0 -1.5708 -> xyz=0 -0.02 0.02 rpy=1.5707963267949 0 -1.5707963267949
- joint joint_3: origin xyz=-0.024 0.195 0 rpy=0 0 1.5708 -> xyz=-0.02 0.2 0 rpy=0 0 1.5707963267949
- joint joint_4: origin xyz=0.02400000035807 -0.0189999998475523 0 rpy=1.5707963267949 0 0 -> xyz=0.0200000000000001 -0.02 0 rpy=1.5707963267949 0 0
- joint joint_5: origin xyz=-0.024 0 0.2085 rpy=-1.5707963267949 0 0 -> xyz=-0.04 0 -0.02 rpy=-1.5707963267949 0 0
- joint joint_6: origin xyz=-0.018999999847552 -0.02400000035807 0 rpy=1.5707963267949 0 -1.5707963267949 -> xyz=-0.02 -0.25 0 rpy=1.5708 0 -1.5708

Commit message: arreglo del urdf nuevo

File: manipulator_final2/urdf/manipulator_final2.urdf (robot description, URDF)
Before this commit: robot manipulator_final2, 7 links, 6 joints
Joints:
- joint joint_1: limit lower=0 upper=3.14 effort=0 velocity=0 -> lower=-1.57 upper=1.57 effort=300 velocity=3
- joint joint_2: limit lower=0 upper=3.14 effort=0 velocity=0 -> lower=-0.78 upper=0.78 effort=300 velocity=3
- joint joint_3: limit lower=0 upper=3.14 effort=0 velocity=0 -> lower=-1.15 upper=2 effort=300 velocity=3
- joint joint_4: limit lower=0 upper=0 effort=3.14 velocity=0 -> lower=-3.14 upper=3.14 effort=200 velocity=3
- joint joint_5: limit lower=0 upper=3.14 effort=0 velocity=0 -> lower=-1.15 upper=2 effort=200 velocity=3
- joint joint_6: limit lower=0 upper=3.14 effort=0 velocity=0 -> lower=-3.14 upper=3.14 effort=200 velocity=3

Commit message: nuevo urdf

File: manipulator_final2/urdf/manipulator_final2.urdf (robot description, URDF)
Before this commit: robot manipulator_final2, 7 links, 6 joints
Links:
- link link_3: mass 0.0569176277607127 -> 0.0569176277607128
- link link_4: mass 0.105070462984835 -> 0.105070462984836
Joints:
- joint joint_5: origin xyz=-0.04 0 -0.02 rpy=-1.5707963267949 0 0 -> xyz=-0.0200000000000001 0 0.21 rpy=-1.5707963267949 0 0
- joint joint_6: origin xyz=-0.02 -0.25 0 rpy=1.5708 0 -1.5708 -> xyz=-0.04 -0.02 0 rpy=1.5707963267949 0 -1.5707963267949
