Commit message: Se reconfiguro todo con xacro, tanto para el robot, para el wolrd y para el ee_marker, en el futuro solo se debe usar otro xacro para cambiar de efector final sin afectar todo el urdf, esto mejora las continuas mejoras que se le puede hacer al proyecto

File: archie_description/urdf/manipulator.urdf (robot description, URDF)
Before this commit: robot manipulator, 8 links, 7 joints
Links:
- link link_6: mass 0.0340927901942582 -> 0.000147831569305485
Joints:
- joint joint_2: origin xyz=0 -0.02 0.02 rpy=1.5707963267949 0 -1.5707963267949 -> xyz=0 -0.024 0.0188 rpy=1.5707963267949 0 -1.5707963267949
- joint joint_3: origin xyz=-0.02 0.2 0 rpy=0 0 1.5707963267949 -> xyz=-0.024 0.195 0 rpy=0 0 1.5707963267949
- joint joint_5: origin xyz=-0.0200000000000001 0 0.21 rpy=-1.5707963267949 0 0 -> xyz=-0.02562 0 0.2075 rpy=-1.5707963267949 0 0
- joint joint_6: origin xyz=-0.04 -0.02 0 rpy=1.5707963267949 0 -1.5707963267949 -> xyz=-0.02 -0.024 0 rpy=1.5707963267949 0 -1.5707963267949

File: archie_description/urdf/manipulator.xacro (robot description, xacro)
@@ -1,4 +1,393 @@
-<?xml version="1.0"?>
-<robot name="manipulator_robot" xmlns:xacro="http://wiki.ros.org/xacro">
-  <xacro:include filename="$(find archie_description)/urdf/manipulator_macro.xacro" />
+<?xml version="1.0" encoding="UTF-8"?>
+<robot xmlns:xacro="http://ros.org/wiki/xacro">
+  <xacro:macro name="manipulator" params="prefix">
+    <link
+      name="${prefix}base_link">
+      <inertial>
+        <origin
+          xyz="5.34102915090199E-06 0.00149611119634719 0.027324411040906"
+          rpy="0 0 0" />
+        <mass
+          value="0.399055600639488" />
+        <inertia
+          ixx="0.101795155"
+          ixy="-0.0000106"
+          ixz="-0.000004255"
+          iyy="0.1049705"
+          iyz="-0.0025166"
+          izz="0.113806134" />
+      </inertial>
+      <visual>
+        <origin
+          xyz="0 0 0"
+          rpy="0 0 0" />
+        <geometry>
+          <mesh
+            filename="package://archie_description/meshes/base_link.STL" />
+        </geometry>
+        <material
+          name="">
+          <color
+            rgba="0.0549 0.4 0.3333 1.0"/>
+        </material>
+      </visual>
+      <collision>
+        <origin
+          xyz="0 0 0"
+          rpy="0 0 0" />
+        <geometry>
+          <mesh
+            filename="package://archie_description/meshes/base_link.STL" />
+        </geometry>
+      </collision>
+    </link>
+    <link
+      name="${prefix}link_1">
+      <inertial>
+        <origin
+          xyz="0.000495971250250975 -0.0119998499605218 0.0192958783777655"
+          rpy="0 0 0" />
+        <mass
+          value="0.102" />
+        <inertia
+          ixx="0.004708"
+          ixy="0.0000362"
+          ixz="-0.0000863"
+          iyy="0.0034761"
+          iyz="-0.0013745"
+          izz="0.0024097" />
+      </inertial>
+      <visual>
+        <origin
+          xyz="0 0 0"
+          rpy="0 0 0" />
+        <geometry>
+          <mesh
+            filename="package://archie_description/meshes/link_1.STL" />
+        </geometry>
+        <material
+          name="">
+          <color
+            rgba="0.09019 0.12549 0.164706 1.0"/>
+        </material>
+      </visual>
+      <collision>
+        <origin
+          xyz="0 0 0"
+          rpy="0 0 0" />
+        <geometry>
+          <mesh
+            filename="package://archie_description/meshes/link_1.STL" />
+        </geometry>
+      </collision>
+    </link>
+    <joint
+      name="${prefix}joint_1"
+      type="revolute">
+      <origin
+        xyz="0 0 0.07"
+        rpy="0 0 3.14159265358979" />
+      <parent
+        link="base_link" />
+      <child
+        link="link_1" />
+      <axis
+        xyz="0 0 1" />
+      <limit
+        lower="-1.57"
+        upper="1.57"
+        effort="300"
+        velocity="3" />
+    </joint>
+    <link
+      name="${prefix}link_2">
+      <inertial>
+        <origin
+          xyz="-0.00375223885247785 0.0986651693444381 3.09623365033344E-07"
+          rpy="0 0 0" />
+        <mass
+          value="0.102283747087815" />
+        <inertia
+          ixx="0.125060728"
+          ixy="0.017650428"
+          ixz="0.000000038"
+          iyy="0.0057453"
+          iyz="-0.00000199"
+          izz="0.1262878" />
+      </inertial>
+      <visual>
+        <origin
+          xyz="-0.004 0.0012 0"
+          rpy="0 0 0" />
+        <geometry>
+          <mesh
+            filename="package://archie_description/meshes/link_2.STL" />
+        </geometry>
+        <material
+          name="">
+          <color
+            rgba="0.1804 0.8 0.4431 1.0"/>
+        </material>
+      </visual>
+      <collision>
+        <origin
+          xyz="-0.004 0.0012 0"
+          rpy="0 0 0" />
+        <geometry>
+          <mesh
+            filename="package://archie_description/meshes/link_2.STL" />
+        </geometry>
+      </collision>
+    </link>
+    <joint
+      name="${prefix}joint_2"
+      type="revolute">
+      <origin
+        xyz="0 -0.024 0.0188"
+        rpy="1.5707963267949 0 -1.5707963267949" />
+      <parent
+        link="link_1" />
+      <child
+        link="link_2" />
+      <axis
+        xyz="0 0 1" />
+      <limit
+        lower="-0.78"
+        upper="0.78"
+        effort="300"
+        velocity="3" />
+    </joint>
+    <link
+      name="${prefix}link_3">
+      <inertial>
+        <origin
+          xyz="0.07998503185917 0.000495971402698678 0.000495878377765527"
+          rpy="0 0 0" />
+        <mass
+          value="0.102" />
+        <inertia
+          ixx="0.004708"
+          ixy="0.0000362"
+          ixz="-0.0000863"
+          iyy="0.0034761"
+          iyz="-0.0013745"
+          izz="0.0024097" />
+      </inertial>
+      <visual>
+        <origin
+          xyz="0.006 0 0"
+          rpy="0 0 0" />
+        <geometry>
+          <mesh
+            filename="package://archie_description/meshes/link_3.STL" />
+        </geometry>
+        <material
+          name="">
+          <color
+            rgba="0.09019 0.12549 0.164706 1.0"/>
+        </material>
+      </visual>
+      <collision>
+        <origin
+          xyz="0.006 0 0"
+          rpy="0 0 0" />
+        <geometry>
+          <mesh
+            filename="package://archie_description/meshes/link_3.STL" />
+        </geometry>
+      </collision>
+    </link>
+    <joint
+      name="${prefix}joint_3"
+      type="revolute">
+      <origin
+        xyz="-0.024 0.195 0"
+        rpy="0 0 1.5707963267949" />
+      <parent
+        link="link_2" />
+      <child
+        link="link_3" />
+      <axis
+        xyz="0 0 1" />
+      <limit
+        lower="-1.15"
+        upper="2"
+        effort="300"
+        velocity="3" />
+    </joint>
+    <link
+      name="${prefix}link_4">
+      <inertial>
+        <origin
+          xyz="-0.0140962967782675 4.33165647224752E-07 0.105115025906125"
+          rpy="0 0 0" />
+        <mass
+          value="0.105070462984836" />
+        <inertia
+          ixx="0.1573144"
+          ixy="0.0195671"
+          ixz="0.0000000040"
+          iyy="0.0051205"
+          iyz="0.0000001350"
+          izz="0.1589789"/>
+      </inertial>
+      <visual>
+        <origin
+          xyz="0 0 0"
+          rpy="0 0 0" />
+        <geometry>
+          <mesh
+            filename="package://archie_description/meshes/link_4.STL" />
+        </geometry>
+        <material
+          name="">
+          <color
+            rgba="0.1804 0.8 0.4431 1.0"/>
+        </material>
+      </visual>
+      <collision>
+        <origin
+          xyz="0 0 0"
+          rpy="0 0 0" />
+        <geometry>
+          <mesh
+            filename="package://archie_description/meshes/link_4.STL" />
+        </geometry>
+      </collision>
+    </link>
+    <joint
+      name="${prefix}joint_4"
+      type="revolute">
+      <origin
+        xyz="0.0200000000000001 -0.02 0"
+        rpy="1.5707963267949 0 0" />
+      <parent
+        link="link_3" />
+      <child
+        link="link_4" />
+      <axis
+        xyz="0 0 1" />
+      <limit
+        lower="-3.14"
+        upper="3.14"
+        effort="200"
+        velocity="3" />
+    </joint>
+    <link
+      name="${prefix}link_5">
+      <inertial>
+        <origin
+          xyz="-0.00570412111171636 -0.00950015024510067 0.000495971250250971"
+          rpy="0 0 0" />
+        <mass
+          value="0.0982" />
+        <inertia
+          ixx="0.004708"
+          ixy="0.0000362"
+          ixz="-0.0000863"
+          iyy="0.0034761"
+          iyz="-0.0013745"
+          izz="0.0024097" />
+      </inertial>
+      <visual>
+        <origin
+          xyz="0.006 -0.0025 0"
+          rpy="0 0 0" />
+        <geometry>
+          <mesh
+            filename="package://archie_description/meshes/link_5.STL" />
+        </geometry>
+        <material
+          name="">
+          <color
+            rgba="0.09019 0.12549 0.164706 1.0"/>
+        </material>
+      </visual>
+      <collision>
+        <origin
+          xyz="0.006 -0.0025 0"
+          rpy="0 0 0" />
+        <geometry>
+          <mesh
+            filename="package://archie_description/meshes/link_5.STL" />
+        </geometry>
+      </collision>
+    </link>
+    <joint
+      name="${prefix}joint_5"
+      type="revolute">
+      <origin
+        xyz="-0.02562 0 0.2075"
+        rpy="-1.5707963267949 0 0" />
+      <parent
+        link="link_4" />
+      <child
+        link="link_5" />
+      <axis
+        xyz="0 0 1" />
+      <limit
+        lower="-1.15"
+        upper="2"
+        effort="200"
+        velocity="3" />
+    </joint>
+    <link
+      name="${prefix}link_6">
+      <inertial>
+        <origin
+          xyz="0.00150005999207131 2.13388833428252E-08 0.0547308096922248"
+          rpy="0 0 0" />
+        <mass
+          value="0.000147831569305485" />
+        <inertia
+          ixx="3.66048153630127E-09"
+          ixy="1.57772181044196E-25"
+          ixz="1.17223439029209E-23"
+          iyy="3.66048153630127E-09"
+          iyz="8.32319653746676E-25"
+          izz="7.31480342388148E-09" />
+      </inertial>
+      <visual>
+        <origin
+          xyz="0 0 0"
+          rpy="0 0 0" />
+        <geometry>
+          <mesh
+            filename="package://archie_description/meshes/link_6.STL" />
+        </geometry>
+        <material
+          name="">
+          <color
+            rgba="0.729411764705882 0.356862745098039 0.0235294117647059 1" />
+        </material>
+      </visual>
+      <collision>
+        <origin
+          xyz="0 0 0"
+          rpy="0 0 0" />
+        <geometry>
+          <mesh
+            filename="package://archie_description/meshes/link_6.STL" />
+        </geometry>
+      </collision>
+    </link>
+    <joint
+      name="${prefix}joint_6"
+      type="revolute">
+      <origin
+        xyz="-0.02 -0.024 0"
+        rpy="1.5707963267949 0 -1.5707963267949" />
+      <parent
+        link="link_5" />
+      <child
+        link="link_6" />
+      <axis
+        xyz="0 0 1" />
+      <limit
+        lower="-3.14"
+        upper="3.14"
+        effort="200"
+        velocity="3" />
+    </joint>
+  </xacro:macro>
 </robot>

File: archie_moveit/config/gazebo_archie.urdf (robot description, URDF)
Before this commit: robot manipulator_robot, 8 links, 7 joints
Links:
- added link ee_marker, mass 0.0340927901942582; collision mesh filename=package://archie_description/meshes/ee_marker.STL; visual mesh filename=package://archie_description/meshes/ee_marker.STL
- link link_6: mass 0.0340927901942582 -> 0.000147831569305485
Joints:
- removed joint world-base_link-fixed
- added joint ee_marker_joint: type fixed, parent link_6, child ee_marker, origin xyz=0 0 0 rpy=0 0 0
- added joint fixed: type fixed, parent world, child base_link, origin xyz=0 0 0 rpy=0 0 0
- joint joint_2: origin xyz=0 -0.02 0.02 rpy=1.5707963267949 0 -1.5707963267949 -> xyz=0 -0.024 0.0188 rpy=1.5707963267949 0 -1.5707963267949
- joint joint_3: origin xyz=-0.02 0.2 0 rpy=0 0 1.5707963267949 -> xyz=-0.024 0.195 0 rpy=0 0 1.5707963267949
- joint joint_5: origin xyz=-0.0200000000000001 0 0.21 rpy=-1.5707963267949 0 0 -> xyz=-0.02562 0 0.2075 rpy=-1.5707963267949 0 0
- joint joint_6: origin xyz=-0.04 -0.02 0 rpy=1.5707963267949 0 -1.5707963267949 -> xyz=-0.02 -0.024 0 rpy=1.5707963267949 0 -1.5707963267949
