Commit message: Matlab file modified to get the mass eigen and damp values wished, also urdf files modified to get a better mass matrix, still there are changes to make

File: archie_description/urdf/manipulator2.urdf (robot description, URDF)
Before this commit: robot manipulator, 8 links, 7 joints
Links:
- link link_6: mass 0.01 -> 0.05

Commit message: Inertias fixed

File: archie_description/urdf/manipulator2.urdf (robot description, URDF)
Before this commit: robot manipulator, 8 links, 7 joints
Links:
- link link_6: mass 0.05 -> 0.1
