Commit message: se realizaron las simulaciones tant en gazebo como en rvz para el pick and place

File: moveit/archie_gripper_moveit/config/gazebo_archie.urdf (robot description, URDF)
Before this commit: robot archie, 12 links, 11 joints
Links:
- link end_effect_point: mass 0.001 -> 0.00001; geometry visual box size=0.0005 0.0005 0.0005
- link garra2_link: mass 0 -> 0.012915
Joints:
- joint garra1_joint: limit lower=0 upper=0.02 effort=100 velocity=0 -> lower=0 upper=0.02 effort=100 velocity=3
- joint garra2_joint: limit lower=-0.02 upper=0 effort=100 velocity=0 -> lower=-0.02 upper=0 effort=100 velocity=3
